File: Models/KiCad/Antenna_Control_System/Antenna_Control_System.kicad_sch (KiCad schematic)
At the start: 21 parts, among them J1 Conn_01x02_Socket, J2 12V IN, J3 USB_C_PLUG, J4 Screw_Terminal_01x07, J5 Conn_Coaxial, J6 Conn_Coaxial, M1 Stepper_Motor_bipolar, SW1 Limit_SW_Push, U1 L7805

Commit message: Revised_README_document
Connections:
- net GNDREF: now also A4.J1 (GND)
- net at A4.3 (NO): no longer A2. (A+)
- net at A1.A3: no longer A4.4 (IN3)
- net at A1.A4: no longer A4.5 (IN4)
- net at A1.D2: now also A4.4 (IN3)
- net at A1.D4: now also A4.5 (IN4)
- net at A1.VIN, C2.1, U1.3 (OUT): now also A4.J3 (JD-VCC)
- new net: A2. (A+), A4.3 (NO)
Changed lines of the file:
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@@
+	)
+	(junction
+		(at 129.54 196.85)
+		(diameter 0)
+		(color 0 0 0 0)
 	)
 	(junction
@@
 	)
 	(junction
+		(at 102.87 148.59)
+		(diameter 0)
+		(color 0 0 0 0)
+	)
+	(junction
 		(at 86.36 187.96)
 		(diameter 0)
@@
 	(wire
 		(pts
+			(xy 113.03 30.48) (xy 114.3 30.48)
+		)
+		(stroke
+			(width 0)
+			(type default)
+		)
+	)
+	(wire
+		(pts
 			(xy 107.95 147.32) (xy 107.95 187.96)
 		)
@@
 	(wire
 		(pts
-			(xy 62.23 45.72) (xy 53.34 45.72)
-		)
-		(stroke
-			(width 0)
-			(type default)
-		)
-	)
-	(wire
-		(pts
 			(xy 128.27 29.21) (xy 129.54 29.21)
 		)
@@
 		(pts
 			(xy 66.04 160.02) (xy 71.12 160.02)
+		)
+		(stroke
+			(width 0)
+			(type default)
+		)
+	)
+	(wire
+		(pts
+			(xy 113.03 25.4) (xy 120.65 25.4)
 		)
 		(stroke
@@
 	(wire
 		(pts
-			(xy 161.29 107.95) (xy 161.29 138.43)
-		)
-		(stroke
-			(width 0)
-			(type default)
-		)
-	)
-	(wire
-		(pts
 			(xy 237.49 87.63) (xy 252.73 87.63)
 		)
@@
 	(wire
 		(pts
-			(xy 160.02 137.16) (xy 53.34 137.16)
-		)
-		(stroke
-			(width 0)
-			(type default)
-		)
-	)
-	(wire
-		(pts
-			(xy 161.29 138.43) (xy 52.07 138.43)
-		)
-		(stroke
-			(width 0)
-			(type default)
-		)
-	)
-	(wire
-		(pts
 			(xy 125.73 44.45) (xy 125.73 17.78)
 		)
@@
 	(wire
 		(pts
+			(xy 129.54 137.16) (xy 129.54 196.85)
+		)
+		(stroke
+			(width 0)
+			(type default)
+		)
+	)
+	(wire
+		(pts
 			(xy 49.53 170.18) (xy 59.69 170.18)
 		)
@@
 	(wire
 		(pts
+			(xy 170.18 142.24) (xy 170.18 144.78)
+		)
+		(stroke
+			(width 0)
+			(type default)
+		)
+	)
+	(wire
+		(pts
 			(xy 147.32 191.77) (xy 147.32 152.4)
 		)
@@
 	(wire
 		(pts
-			(xy 53.34 45.72) (xy 53.34 137.16)
-		)
-		(stroke
-			(width 0)
-			(type default)
-		)
-	)
-	(wire
-		(pts
 			(xy 59.69 91.44) (xy 62.23 91.44)
 		)
@@
 	(wire
 		(pts
+			(xy 129.54 196.85) (xy 156.21 196.85)
+		)
+		(stroke
+			(width 0)
+			(type default)
+		)
+	)
+	(wire
+		(pts
 			(xy 195.58 92.71) (xy 215.9 92.71)
 		)
@@
 		(pts
 			(xy 59.69 196.85) (xy 127 196.85)
+		)
+		(stroke
+			(width 0)
+			(type default)
+		)
+	)
+	(wire
+		(pts
+			(xy 120.65 105.41) (xy 170.18 105.41)
 		)
 		(stroke
@@
 	(wire
 		(pts
-			(xy 62.23 43.18) (xy 52.07 43.18)
-		)
-		(stroke
-			(width 0)
-			(type default)
-		)
-	)
-	(wire
-		(pts
 			(xy 71.12 180.34) (xy 71.12 187.96)
 		)
@@
 	(wire
 		(pts
-			(xy 52.07 43.18) (xy 52.07 138.43)
-		)
-		(stroke
-			(width 0)
-			(type default)
-		)
-	)
-	(wire
-		(pts
 			(xy 57.15 81.28) (xy 57.15 142.24)
 		)
@@
 	(wire
 		(pts
-			(xy 160.02 105.41) (xy 160.02 137.16)
-		)
-		(stroke
-			(width 0)
-			(type default)
-		)
-	)
-	(wire
-		(pts
 			(xy 219.71 31.75) (xy 219.71 57.15)
 		)
@@
 	(wire
 		(pts
+			(xy 170.18 144.78) (xy 102.87 144.78)
+		)
+		(stroke
+			(width 0)
+			(type default)
+		)
+	)
+	(wire
+		(pts
 			(xy 33.02 191.77) (xy 147.32 191.77)
 		)
@@
 	(wire
 		(pts
+			(xy 170.18 137.16) (xy 129.54 137.16)
+		)
+		(stroke
+			(width 0)
+			(type default)
+		)
+	)
+	(wire
+		(pts
 			(xy 219.71 57.15) (xy 237.49 57.15)
 		)
@@
 	(wire
 		(pts
+			(xy 102.87 144.78) (xy 102.87 148.59)
+		)
+		(stroke
+			(width 0)
+			(type default)
+		)
+	)
+	(wire
+		(pts
 			(xy 121.92 36.83) (xy 129.54 36.83)
 		)
@@
 	(wire
 		(pts
+			(xy 114.3 30.48) (xy 114.3 107.95)
+		)
+		(stroke
+			(width 0)
+			(type default)
+		)
+	)
+	(wire
+		(pts
 			(xy 62.23 40.64) (xy 50.8 40.64)
 		)
@@
 	(wire
 		(pts
-			(xy 170.18 105.41) (xy 160.02 105.41)
+			(xy 114.3 107.95) (xy 170.18 107.95)
 		)
 		(stroke
@@
 	(wire
 		(pts
-			(xy 127 196.85) (xy 156.21 196.85)
+			(xy 127 196.85) (xy 129.54 196.85)
 		)
 		(stroke
@@
 	(wire
 		(pts
-			(xy 170.18 107.95) (xy 161.29 107.95)
-		)
-		(stroke
-			(width 0)
-			(type default)
-		)
-	)
-	(wire
-		(pts
 			(xy 25.4 120.65) (xy 25.4 124.46)
 		)
@@
 		)
 		(stroke
+			(width 0)
+			(type default)
+		)
+	)
+	(wire
+		(pts
+			(xy 120.65 25.4) (xy 120.65 105.41)
+		)
+		(stroke

Commit message: Revised Schematic
Parts:
- removed J4: Screw_Terminal_01x07, symbol Connector:Screw_Terminal_01x07
Connections:
- net at L2.Signal: now also A4.2 (COM)
- net at A4.3 (NO): no longer A2. (A+)
- new net: A2. (A+), A4.3 (NO)
- now unconnected: A4.2 (COM), A4.2 (COM), A4.2 (COM), A4.2 (COM)
